Commit message: Added multiple bebop support

File: bebop_gazebo/urdf/bebop_aerodynamics.gazebo.xacro (robot description, xacro)
@@ -1,4 +1,6 @@
 <?xml version="1.0"?>
 <robot xmlns:xacro="http://www.ros.org/wiki/xacro">
+<xacro:arg name="prefix" default=""/>
+  <xacro:property name= "prefix" value="$(arg prefix)"/>
   <!-- Quadrotor Aerodynamics Plugin -->
   <xacro:macro name="bebop_aerodynamics">
@@ -7,6 +9,6 @@
         <alwaysOn>true</alwaysOn>
         <updateRate>0.0</updateRate>
-        <bodyName>base_link</bodyName>
-        <frameId>$(arg base_link_frame)</frameId>
+        <bodyName>${prefix}base_link</bodyName>
+        <frameId>${prefix}base_link</frameId>
       </plugin>
     </gazebo>

File: bebop_gazebo/urdf/bebop_base.urdf.xacro (robot description, xacro)
@@ -11,7 +11,9 @@
   <xacro:property name="tilt_vel" value="2.0" />
   <xacro:property name="joint_effort" value="50" />
+  <xacro:arg name="prefix" default=""/>
+  <xacro:property name= "prefix" value="$(arg prefix)"/>
   <!-- Main quadrotor link -->
   <xacro:macro name="bebop_base_macro">
-    <link name="base_link">
+    <link name="${prefix}base_link">
       <inertial>
         <mass value="0.399" />
@@ -23,4 +25,5 @@
         <origin xyz="0 0 0" rpy="0 0 0" />
         <geometry>
+          <!-- <mesh filename="package://bebop_gazebo/meshes/bebop_model.stl" scale="4 4 4"/> -->
           <mesh filename="package://bebop_gazebo/meshes/bebop_model.stl"/>
         </geometry>
@@ -36,34 +39,37 @@
       </collision>
     </link>
-    <link name="camera_base_link"></link>
-    <link name="camera_pan_link"></link>
-    <link name="camera_tilt_link"></link>
-    <link name="camera_optical"></link>
-    <joint name="base_link_joint" type="fixed">
+    <link name="${prefix}camera_base_link"></link>
+    <link name="${prefix}camera_pan_link"></link>
+    <link name="${prefix}camera_tilt_link"></link>
+    <link name="${prefix}camera_optical"></link>
+    <joint name="${prefix}base_link_joint" type="fixed">
       <origin xyz="${camera_offset_len} 0 ${camera_offset_ver}" rpy="0 0 0" />
-      <parent link="base_link"/>
-      <child link="camera_base_link" />
+      <parent link="${prefix}base_link"/>
+      <child link="${prefix}camera_base_link" />
     </joint>
-    <joint name="camera_pan_joint" type="revolute">
+    <joint name="${prefix}camera_pan_joint" type="revolute">
       <origin xyz="0 0 0" rpy="0 0 0" />
-      <parent link="camera_base_link" />
-      <child link="camera_pan_link" />
+      <parent link="${prefix}camera_base_link" />
+      <child link="${prefix}camera_pan_link" />
       <axis xyz="0 0 1" />
       <limit lower="${-pan_range}" upper="${pan_range}"
         effort="${joint_effort}" velocity="${pan_vel}" />
     </joint>
-    <joint name="camera_tilt_joint" type="revolute">
+    <joint name="${prefix}camera_tilt_joint" type="revolute">
       <origin xyz="0 0 0" rpy="0 0 0" />
-      <parent link="camera_pan_link" />
-      <child link="camera_tilt_link" />
+      <parent link="${prefix}camera_pan_link" />
+      <child link="${prefix}camera_tilt_link" />
       <axis xyz="0 1 0" />
       <limit lower="${-tilt_range}" upper="${tilt_range}"
         effort="${joint_effort}" velocity="${tilt_vel}" />
     </joint>
-    <joint name="camera_optical_joint" type="fixed">
+    <joint name="${prefix}camera_optical_joint" type="fixed">
       <origin xyz="0 0 0" rpy="${-pi/2} 0 ${-pi/2}" />
-      <parent link="camera_tilt_link" />
-      <child link="camera_optical" />
+      <parent link="${prefix}camera_tilt_link" />
+      <child link="${prefix}camera_optical" />
     </joint>
+     <gazebo reference="${prefix}base_link">
+      <material>Gazebo/Black</material>
+    </gazebo>
   </xacro:macro>
 </robot>

File: bebop_gazebo/urdf/bebop_plugins.gazebo.xacro (robot description, xacro)
@@ -2,5 +2,4 @@
 <robot xmlns:xacro="http://www.ros.org/wiki/xacro">
   <xacro:arg name="world_frame" default="world"/>
-  <xacro:arg name="base_link_frame" default="base_link"/>
   <xacro:include filename="$(find bebop_gazebo)/urdf/bebop_sensors.gazebo.xacro" />
   <xacro:include filename="$(find bebop_gazebo)/urdf/bebop_controller.gazebo.xacro" />

File: bebop_gazebo/urdf/bebop_propulsion.gazebo.xacro (robot description, xacro)
@@ -7,6 +7,6 @@
         <alwaysOn>true</alwaysOn>
         <updateRate>0.0</updateRate>
-        <bodyName>base_link</bodyName>
-        <frameId>$(arg base_link_frame)</frameId>
+        <bodyName>${prefix}base_link</bodyName>
+        <frameId>${prefix}base_link</frameId>
         <controlRate>100.0</controlRate>
         <controlTolerance>0.01</controlTolerance>

File: bebop_gazebo/urdf/bebop_sensors.gazebo.xacro (robot description, xacro)
@@ -1,9 +1,11 @@
 <?xml version="1.0"?>
 <robot xmlns:xacro="http://www.ros.org/wiki/xacro">
+<xacro:arg name="prefix" default=""/>
+<xacro:property name= "prefix" value="$(arg prefix)"/>
   <!-- Quadrotor Sensor Plugins -->
   <xacro:macro name="bebop_sensors">
-    <gazebo reference="camera_base_link">
+    <gazebo reference="${prefix}camera_base_link">
       <sensor type="camera" name="bebop_camera_sensor">
-        <update_rate>30.0</update_rate>
+        <update_rate>50.0</update_rate>
         <camera name="front">
           <horizontal_fov>1.570796</horizontal_fov>
@@ -19,20 +21,21 @@
         </camera>
         <plugin name="bebop_camera_controller" filename="libgazebo_ros_camera.so">
-        <cameraName>/bebop/camera</cameraName>
+        <cameraName>${prefix}camera</cameraName>
           <alwaysOn>true</alwaysOn>
-          <updateRate>30.0</updateRate>
-          <imageTopicName>/bebop/image_raw</imageTopicName>
-          <cameraInfoTopicName>/bebop/camera_info</cameraInfoTopicName>
-          <frameName>camera_optical</frameName>
+          <updateRate>50.0</updateRate>
+          <imageTopicName>image_raw</imageTopicName>
+          <cameraInfoTopicName>camera_info</cameraInfoTopicName>
+          <frameName>${prefix}camera_optical</frameName>
         </plugin>
       </sensor>
     </gazebo>
+    <xacro:property name="deg_to_rad" value="0.01745329251994329577" />
         <gazebo>
           <plugin name="bebop_gps_sim" filename="libhector_gazebo_ros_gps.so">
             <updateRate>4.0</updateRate>
-            <bodyName>base_link</bodyName>
-            <frameId>$(arg base_link_frame)</frameId>
-            <topicName>/bebop/fix</topicName>
-            <velocityTopicName>/bebop/fix_velocity</velocityTopicName>
+            <bodyName>${prefix}base_link</bodyName>
+            <frameId>${prefix}base_link</frameId>
+            <topicName>fix</topicName>
+            <velocityTopicName>fix_velocity</velocityTopicName>
             <referenceLatitude>37.9707</referenceLatitude>
             <referenceLongitude>23.7294</referenceLongitude>
@@ -44,6 +47,6 @@
           <plugin name="bebop_groundtruth_sim" filename="libgazebo_ros_p3d.so">
             <updateRate>100.0</updateRate>
-            <bodyName>base_link</bodyName>
-            <topicName>/bebop/odom</topicName>
+            <bodyName>${prefix}base_link</bodyName>
+            <topicName>odom</topicName>
             <gaussianNoise>0.0</gaussianNoise>
             <frameName>$(arg world_frame)</frameName>

Commit message: bebop_gazebo original package

File: bebop_gazebo/urdf/bebop_aerodynamics.gazebo.xacro (robot description, xacro)
@@ -1,6 +1,4 @@
 <?xml version="1.0"?>
 <robot xmlns:xacro="http://www.ros.org/wiki/xacro">
-<xacro:arg name="prefix" default=""/>
-  <xacro:property name= "prefix" value="$(arg prefix)"/>
   <!-- Quadrotor Aerodynamics Plugin -->
   <xacro:macro name="bebop_aerodynamics">
@@ -9,6 +7,6 @@
         <alwaysOn>true</alwaysOn>
         <updateRate>0.0</updateRate>
-        <bodyName>${prefix}base_link</bodyName>
-        <frameId>${prefix}base_link</frameId>
+        <bodyName>base_link</bodyName>
+        <frameId>$(arg base_link_frame)</frameId>
       </plugin>
     </gazebo>

File: bebop_gazebo/urdf/bebop_base.urdf.xacro (robot description, xacro)
@@ -11,9 +11,7 @@
   <xacro:property name="tilt_vel" value="2.0" />
   <xacro:property name="joint_effort" value="50" />
-  <xacro:arg name="prefix" default=""/>
-  <xacro:property name= "prefix" value="$(arg prefix)"/>
   <!-- Main quadrotor link -->
   <xacro:macro name="bebop_base_macro">
-    <link name="${prefix}base_link">
+    <link name="base_link">
       <inertial>
         <mass value="0.399" />
@@ -25,5 +23,4 @@
         <origin xyz="0 0 0" rpy="0 0 0" />
         <geometry>
-          <!-- <mesh filename="package://bebop_gazebo/meshes/bebop_model.stl" scale="4 4 4"/> -->
           <mesh filename="package://bebop_gazebo/meshes/bebop_model.stl"/>
         </geometry>
@@ -39,37 +36,34 @@
       </collision>
     </link>
-    <link name="${prefix}camera_base_link"></link>
-    <link name="${prefix}camera_pan_link"></link>
-    <link name="${prefix}camera_tilt_link"></link>
-    <link name="${prefix}camera_optical"></link>
-    <joint name="${prefix}base_link_joint" type="fixed">
+    <link name="camera_base_link"></link>
+    <link name="camera_pan_link"></link>
+    <link name="camera_tilt_link"></link>
+    <link name="camera_optical"></link>
+    <joint name="base_link_joint" type="fixed">
       <origin xyz="${camera_offset_len} 0 ${camera_offset_ver}" rpy="0 0 0" />
-      <parent link="${prefix}base_link"/>
-      <child link="${prefix}camera_base_link" />
+      <parent link="base_link"/>
+      <child link="camera_base_link" />
     </joint>
-    <joint name="${prefix}camera_pan_joint" type="revolute">
+    <joint name="camera_pan_joint" type="revolute">
       <origin xyz="0 0 0" rpy="0 0 0" />
-      <parent link="${prefix}camera_base_link" />
-      <child link="${prefix}camera_pan_link" />
+      <parent link="camera_base_link" />
+      <child link="camera_pan_link" />
       <axis xyz="0 0 1" />
       <limit lower="${-pan_range}" upper="${pan_range}"
         effort="${joint_effort}" velocity="${pan_vel}" />
     </joint>
-    <joint name="${prefix}camera_tilt_joint" type="revolute">
+    <joint name="camera_tilt_joint" type="revolute">
       <origin xyz="0 0 0" rpy="0 0 0" />
-      <parent link="${prefix}camera_pan_link" />
-      <child link="${prefix}camera_tilt_link" />
+      <parent link="camera_pan_link" />
+      <child link="camera_tilt_link" />
       <axis xyz="0 1 0" />
       <limit lower="${-tilt_range}" upper="${tilt_range}"
         effort="${joint_effort}" velocity="${tilt_vel}" />
     </joint>
-    <joint name="${prefix}camera_optical_joint" type="fixed">
+    <joint name="camera_optical_joint" type="fixed">
       <origin xyz="0 0 0" rpy="${-pi/2} 0 ${-pi/2}" />
-      <parent link="${prefix}camera_tilt_link" />
-      <child link="${prefix}camera_optical" />
+      <parent link="camera_tilt_link" />
+      <child link="camera_optical" />
     </joint>
-     <gazebo reference="${prefix}base_link">
-      <material>Gazebo/Black</material>
-    </gazebo>
   </xacro:macro>
 </robot>

File: bebop_gazebo/urdf/bebop_plugins.gazebo.xacro (robot description, xacro)
@@ -2,4 +2,5 @@
 <robot xmlns:xacro="http://www.ros.org/wiki/xacro">
   <xacro:arg name="world_frame" default="world"/>
+  <xacro:arg name="base_link_frame" default="base_link"/>
   <xacro:include filename="$(find bebop_gazebo)/urdf/bebop_sensors.gazebo.xacro" />
   <xacro:include filename="$(find bebop_gazebo)/urdf/bebop_controller.gazebo.xacro" />

File: bebop_gazebo/urdf/bebop_propulsion.gazebo.xacro (robot description, xacro)
@@ -7,6 +7,6 @@
         <alwaysOn>true</alwaysOn>
         <updateRate>0.0</updateRate>
-        <bodyName>${prefix}base_link</bodyName>
-        <frameId>${prefix}base_link</frameId>
+        <bodyName>base_link</bodyName>
+        <frameId>$(arg base_link_frame)</frameId>
         <controlRate>100.0</controlRate>
         <controlTolerance>0.01</controlTolerance>

File: bebop_gazebo/urdf/bebop_sensors.gazebo.xacro (robot description, xacro)
@@ -1,12 +1,9 @@
 <?xml version="1.0"?>
 <robot xmlns:xacro="http://www.ros.org/wiki/xacro">
-<xacro:arg name="prefix" default=""/>
-<xacro:property name= "prefix" value="$(arg prefix)"/>
-<xacro:property name="deg_to_rad" value="0.01745329251994329577" />
   <!-- Quadrotor Sensor Plugins -->
   <xacro:macro name="bebop_sensors">
-    <!-- <gazebo reference="${prefix}camera_base_link">
+    <gazebo reference="camera_base_link">
       <sensor type="camera" name="bebop_camera_sensor">
-        <update_rate>50.0</update_rate>
+        <update_rate>30.0</update_rate>
         <camera name="front">
           <horizontal_fov>1.570796</horizontal_fov>
@@ -22,148 +19,20 @@
         </camera>
         <plugin name="bebop_camera_controller" filename="libgazebo_ros_camera.so">
-        <cameraName>${prefix}camera</cameraName>
+        <cameraName>/bebop/camera</cameraName>
           <alwaysOn>true</alwaysOn>
-          <updateRate>50.0</updateRate>
-          <imageTopicName>image_raw</imageTopicName>
-          <cameraInfoTopicName>camera_info</cameraInfoTopicName>
-          <frameName>${prefix}camera_optical</frameName>
+          <updateRate>30.0</updateRate>
+          <imageTopicName>/bebop/image_raw</imageTopicName>
+          <cameraInfoTopicName>/bebop/camera_info</cameraInfoTopicName>
+          <frameName>camera_optical</frameName>
         </plugin>
       </sensor>
-    </gazebo> -->
- <gazebo reference="${prefix}camera_base_link">
-      <self_collide>0</self_collide>
-      <enable_wind>0</enable_wind>
-      <kinematic>0</kinematic>
-      <gravity>1</gravity>
-      <!--<mu>1</mu>-->
-      <mu2>1</mu2>
-      <fdir1>0 0 0</fdir1>
-      <!--<slip1>0</slip1>
-      <slip2>0</slip2>-->
-      <kp>1e+13</kp>
-      <kd>1</kd>
-      <!--<max_vel>0.01</max_vel>
-      <min_depth>0</min_depth>-->
-      <sensor name="color" type="camera">
-        <camera name="real_sense">
-          <horizontal_fov>${69.4*deg_to_rad}</horizontal_fov>
-          <image>
-            <width>640</width>
-            <height>480</height>
-            <format>RGB_INT8</format>
-          </image>
-          <clip>
-            <near>0.1</near>
-            <far>100</far>
-          </clip>
-          <noise>
-            <type>gaussian</type>
-            <mean>0.0</mean>
-            <stddev>0.007</stddev>
-          </noise>
-        </camera>
-        <always_on>1</always_on>
-        <update_rate>30</update_rate>
-        <visualize>1</visualize>
-      </sensor>
-      <sensor name="ired1" type="camera">
-        <camera name="real_sense">
-          <horizontal_fov>${85.2*deg_to_rad}</horizontal_fov>
-          <image>
-            <width>1280</width>
-            <height>720</height>
-            <format>L_INT8</format>
-          </image>
-          <clip>
-            <near>0.1</near>
-            <far>100</far>
-          </clip>
-          <noise>
-            <type>gaussian</type>
-            <mean>0.0</mean>
-            <stddev>0.05</stddev>
-          </noise>
-        </camera>
-        <always_on>1</always_on>
-        <update_rate>90</update_rate>
-        <visualize>0</visualize>
-      </sensor>
-      <sensor name="ired2" type="camera">
-        <camera name="real_sense">
-          <horizontal_fov>${85.2*deg_to_rad}</horizontal_fov>
-          <image>
-            <width>1280</width>
-            <height>720</height>
-            <format>L_INT8</format>
-          </image>
-          <clip>
-            <near>0.1</near>
-            <far>100</far>
-          </clip>
-          <noise>
-            <type>gaussian</type>
-            <mean>0.0</mean>
-            <stddev>0.05</stddev>
-          </noise>
-        </camera>
-        <always_on>1</always_on>
-        <update_rate>90</update_rate>
-        <visualize>0</visualize>
-      </sensor>
-      <sensor name="depth" type="depth">
-        <camera name="real_sense">
-          <horizontal_fov>${85.2*deg_to_rad}</horizontal_fov>
-          <image>
-            <width>1280</width>
-            <height>720</height>
-          </image>
-          <clip>
-            <near>0.1</near>
-            <far>100</far>
-          </clip>
-          <noise>
-            <type>gaussian</type>
-            <mean>0.0</mean>
-            <stddev>0.100</stddev>
-          </noise>
-        </camera>
-        <always_on>1</always_on>
-        <update_rate>90</update_rate>
-        <visualize>0</visualize>
-      </sensor>
-    </gazebo>
-    <gazebo>
-      <plugin name="realsense" filename="librealsense_gazebo_plugin.so">
-        <!-- <prefix>${camera_name}</prefix> -->
-        <depthUpdateRate>30.0</depthUpdateRate>
-        <colorUpdateRate>30.0</colorUpdateRate>
-        <infraredUpdateRate>30.0</infraredUpdateRate>
-        <depthTopicName>depth/image_raw</depthTopicName>
-        <depthCameraInfoTopicName>depth/camera_info</depthCameraInfoTopicName>
-        <colorTopicName>color/image_raw</colorTopicName>
-        <colorCameraInfoTopicName>color/camera_info</colorCameraInfoTopicName>
-        <infrared1TopicName>infra1/image_raw</infrared1TopicName>
-        <infrared1CameraInfoTopicName>infra1/camera_info</infrared1CameraInfoTopicName>
-        <infrared2TopicName>infra2/image_raw</infrared2TopicName>
-        <infrared2CameraInfoTopicName>infra2/camera_info</infrared2CameraInfoTopicName>
-        <colorOpticalframeName>${prefix}camera_optical</colorOpticalframeName>
-        <depthOpticalframeName>${prefix}camera_optical</depthOpticalframeName>
-        <infrared1OpticalframeName>${prefix}camera_optical</infrared1OpticalframeName>
-        <infrared2OpticalframeName>${prefix}camera_optical</infrared2OpticalframeName>
-        <rangeMinDepth>0.2</rangeMinDepth>
-        <rangeMaxDepth>10.0</rangeMaxDepth>
-        <pointCloud>true</pointCloud>
-        <pointCloudTopicName>depth/color/points</pointCloudTopicName>
-        <pointCloudCutoff>0.25</pointCloudCutoff>
-        <pointCloudCutoffMax>9.0</pointCloudCutoffMax>
-      </plugin>
     </gazebo>
         <gazebo>
           <plugin name="bebop_gps_sim" filename="libhector_gazebo_ros_gps.so">
             <updateRate>4.0</updateRate>
-            <bodyName>${prefix}base_link</bodyName>
-            <frameId>${prefix}base_link</frameId>
-            <topicName>fix</topicName>
-            <velocityTopicName>fix_velocity</velocityTopicName>
+            <bodyName>base_link</bodyName>
+            <frameId>$(arg base_link_frame)</frameId>
+            <topicName>/bebop/fix</topicName>
+            <velocityTopicName>/bebop/fix_velocity</velocityTopicName>
             <referenceLatitude>37.9707</referenceLatitude>
             <referenceLongitude>23.7294</referenceLongitude>
@@ -175,6 +44,6 @@
           <plugin name="bebop_groundtruth_sim" filename="libgazebo_ros_p3d.so">
             <updateRate>100.0</updateRate>
-            <bodyName>${prefix}base_link</bodyName>
-            <topicName>odom</topicName>
+            <bodyName>base_link</bodyName>
+            <topicName>/bebop/odom</topicName>
             <gaussianNoise>0.0</gaussianNoise>
             <frameName>$(arg world_frame)</frameName>
