Commit message: changed the color of bebop and added Yaw argument to spawn launch file

File: bebop_gazebo/urdf/bebop_base.urdf.xacro (robot description, xacro)
@@ -66,4 +66,7 @@
       <child link="camera_optical" />
     </joint>
+    <gazebo reference="base_link">
+      <material>Gazebo/Black</material>
+    </gazebo>
   </xacro:macro>
 </robot>
