Commit message: added lidar to bebop

File: bebop_gazebo/urdf/bebop.urdf.xacro (robot description, xacro)
@@ -2,8 +2,41 @@
 <robot
   name="quadrotor"
-  xmlns:xacro="http://www.ros.org/wiki/xacro"
->
+  xmlns:xacro="http://www.ros.org/wiki/xacro">
     <!-- Included URDF Files -->
     <xacro:include filename="$(find bebop_gazebo)/urdf/bebop_base.urdf.xacro" />
     <xacro:bebop_base_macro />
+    <xacro:property name="laser_size_x" value="0.03"/>
+    <xacro:property name="laser_size_y" value="0.03"/>
+    <xacro:property name="laser_size_z" value="0.04"/>
+    <xacro:property name="laser_origin_x" value="0.0"/>
+    <xacro:property name="laser_origin_y" value="0"/>
+    <xacro:property name="laser_origin_z" value="0.08"/>
+  <xacro:property name="base_radius" value="0.05"/>
+  <xacro:property name="base_height" value="0.05"/>
+  <xacro:property name="laz_radius" value="0.04"/>
+  <xacro:property name="laz_height" value="0.1"/>
+  <!--Laser Scan-->
+  <link name="sensor_laser">
+    <visual>
+      <geometry>
+        <mesh filename="package://bebop_gazebo/meshes/hokuyo.dae"/>
+        <!--box size="${laser_size_x} ${laser_size_y} ${laser_size_z}"/-->
+      </geometry>
+      <material name="blue"/>
+    </visual>
+    <collision>
+      <geometry>
+        <box size="${laser_size_x} ${laser_size_y} ${laser_size_z}"/>
+      </geometry>
+    </collision>
+    <inertial>
+      <mass value="0.00000000001"/>
+      <inertia ixx="${(1/12) * 0.1 * (3 * base_radius * base_radius + base_height * base_height)}" ixy="0" ixz="0" iyy="${(1/12) * 0.1 * (3 * base_radius * base_radius + base_height * base_height)}" iyz="0" izz="${(1/2) * 0.1 * base_radius * base_radius}"/>
+    </inertial>
+  </link>
+  <joint name="sensor_laser_joint" type="fixed">
+    <origin xyz="${laser_origin_x} ${laser_origin_y} ${laser_origin_z}" rpy="0 0 0" />
+    <parent link="base_link"/>
+    <child link="sensor_laser" />
+  </joint>
 </robot>

File: bebop_gazebo/urdf/bebop_sensors.gazebo.xacro (robot description, xacro)
@@ -50,4 +50,35 @@
           </plugin>
         </gazebo>
+    <gazebo reference="sensor_laser">
+      <sensor type="ray" name="head_hokuyo_sensor">
+      <pose>0 0 0 0 0 0</pose>
+      <visualize>false</visualize>
+      <update_rate>40</update_rate>
+      <ray>
+        <scan>
+          <horizontal>
+            <samples>360</samples>
+            <resolution>1</resolution>
+            <min_angle>-3.14</min_angle>
+            <max_angle>3.14</max_angle>
+          </horizontal>
+        </scan>
+        <range>
+          <min>0.10</min>
+          <max>10.0</max>
+          <resolution>0.01</resolution>
+        </range>
+        <noise>
+          <type>gaussian</type>
+          <mean>0.0</mean>
+          <stddev>0.01</stddev>
+        </noise>
+      </ray>
+      <plugin name="gazebo_ros_head_hokuyo_controller" filename="libgazebo_ros_laser.so">
+        <topicName>/bebop/laser_scan</topicName>
+        <frameName>sensor_laser</frameName>
+      </plugin>
+    </sensor>
+  </gazebo>
   </xacro:macro>
 </robot>

Commit message: added support for multiple bebops

File: bebop_gazebo/urdf/bebop.urdf.xacro (robot description, xacro)
@@ -16,6 +16,8 @@
   <xacro:property name="laz_radius" value="0.04"/>
   <xacro:property name="laz_height" value="0.1"/>
+  <xacro:arg name="prefix" default=""/>
+  <xacro:property name= "prefix" value="$(arg prefix)"/>
   <!--Laser Scan-->
-  <link name="sensor_laser">
+  <link name="${prefix}sensor_laser">
     <visual>
       <geometry>
@@ -35,8 +37,8 @@
     </inertial>
   </link>
-  <joint name="sensor_laser_joint" type="fixed">
+  <joint name="bebop_sensor_laser_joint" type="fixed">
     <origin xyz="${laser_origin_x} ${laser_origin_y} ${laser_origin_z}" rpy="0 0 0" />
-    <parent link="base_link"/>
-    <child link="sensor_laser" />
+    <parent link="${prefix}base_link"/>
+    <child link="${prefix}sensor_laser" />
   </joint>
 </robot>

File: bebop_gazebo/urdf/bebop_base.urdf.xacro (robot description, xacro)
@@ -11,7 +11,9 @@
   <xacro:property name="tilt_vel" value="2.0" />
   <xacro:property name="joint_effort" value="50" />
+  <xacro:arg name="prefix" default=""/>
+  <xacro:property name= "prefix" value="$(arg prefix)"/>
   <!-- Main quadrotor link -->
   <xacro:macro name="bebop_base_macro">
-    <link name="base_link">
+    <link name="${prefix}base_link">
       <inertial>
         <mass value="0.399" />
@@ -36,35 +38,35 @@
       </collision>
     </link>
-    <link name="camera_base_link"></link>
-    <link name="camera_pan_link"></link>
-    <link name="camera_tilt_link"></link>
-    <link name="camera_optical"></link>
-    <joint name="base_link_joint" type="fixed">
+    <link name="${prefix}camera_base_link"></link>
+    <link name="${prefix}camera_pan_link"></link>
+    <link name="${prefix}camera_tilt_link"></link>
+    <link name="${prefix}camera_optical"></link>
+    <joint name="${prefix}base_link_joint" type="fixed">
       <origin xyz="${camera_offset_len} 0 ${camera_offset_ver}" rpy="0 0 0" />
-      <parent link="base_link"/>
-      <child link="camera_base_link" />
+      <parent link="${prefix}base_link"/>
+      <child link="${prefix}camera_base_link" />
     </joint>
-    <joint name="camera_pan_joint" type="revolute">
+    <joint name="${prefix}camera_pan_joint" type="revolute">
       <origin xyz="0 0 0" rpy="0 0 0" />
-      <parent link="camera_base_link" />
-      <child link="camera_pan_link" />
+      <parent link="${prefix}camera_base_link" />
+      <child link="${prefix}camera_pan_link" />
       <axis xyz="0 0 1" />
       <limit lower="${-pan_range}" upper="${pan_range}"
         effort="${joint_effort}" velocity="${pan_vel}" />
     </joint>
-    <joint name="camera_tilt_joint" type="revolute">
+    <joint name="${prefix}camera_tilt_joint" type="revolute">
       <origin xyz="0 0 0" rpy="0 0 0" />
-      <parent link="camera_pan_link" />
-      <child link="camera_tilt_link" />
+      <parent link="${prefix}camera_pan_link" />
+      <child link="${prefix}camera_tilt_link" />
       <axis xyz="0 1 0" />
       <limit lower="${-tilt_range}" upper="${tilt_range}"
         effort="${joint_effort}" velocity="${tilt_vel}" />
     </joint>
-    <joint name="camera_optical_joint" type="fixed">
+    <joint name="${prefix}camera_optical_joint" type="fixed">
       <origin xyz="0 0 0" rpy="${-pi/2} 0 ${-pi/2}" />
-      <parent link="camera_tilt_link" />
-      <child link="camera_optical" />
+      <parent link="${prefix}camera_tilt_link" />
+      <child link="${prefix}camera_optical" />
     </joint>
-    <gazebo reference="base_link">
+    <gazebo reference="${prefix}base_link">
       <material>Gazebo/Black</material>
     </gazebo>

File: bebop_gazebo/urdf/bebop_sensors.gazebo.xacro (robot description, xacro)
@@ -1,9 +1,12 @@
 <?xml version="1.0"?>
 <robot xmlns:xacro="http://www.ros.org/wiki/xacro">
+<xacro:arg name="prefix" default=""/>
+<xacro:property name= "prefix" value="$(arg prefix)"/>
+<xacro:property name="deg_to_rad" value="0.01745329251994329577" />
   <!-- Quadrotor Sensor Plugins -->
   <xacro:macro name="bebop_sensors">
-    <gazebo reference="camera_base_link">
+    <gazebo reference="${prefix}camera_base_link">
       <sensor type="camera" name="bebop_camera_sensor">
-        <update_rate>30.0</update_rate>
+        <update_rate>50.0</update_rate>
         <camera name="front">
           <horizontal_fov>1.570796</horizontal_fov>
@@ -19,10 +22,10 @@
         </camera>
         <plugin name="bebop_camera_controller" filename="libgazebo_ros_camera.so">
-        <cameraName>/bebop/camera</cameraName>
+        <cameraName>${prefix}camera</cameraName>
           <alwaysOn>true</alwaysOn>
-          <updateRate>30.0</updateRate>
-          <imageTopicName>/bebop/image_raw</imageTopicName>
-          <cameraInfoTopicName>/bebop/camera_info</cameraInfoTopicName>
-          <frameName>camera_optical</frameName>
+          <updateRate>50.0</updateRate>
+          <imageTopicName>image_raw</imageTopicName>
+          <cameraInfoTopicName>camera_info</cameraInfoTopicName>
+          <frameName>${prefix}camera_optical</frameName>
         </plugin>
       </sensor>
@@ -31,8 +34,8 @@
           <plugin name="bebop_gps_sim" filename="libhector_gazebo_ros_gps.so">
             <updateRate>4.0</updateRate>
-            <bodyName>base_link</bodyName>
-            <frameId>$(arg base_link_frame)</frameId>
-            <topicName>/bebop/fix</topicName>
-            <velocityTopicName>/bebop/fix_velocity</velocityTopicName>
+            <bodyName>${prefix}base_link</bodyName>
+            <frameId>${prefix}base_link</frameId>
+            <topicName>fix</topicName>
+            <velocityTopicName>fix_velocity</velocityTopicName>
             <referenceLatitude>37.9707</referenceLatitude>
             <referenceLongitude>23.7294</referenceLongitude>
@@ -44,11 +47,11 @@
           <plugin name="bebop_groundtruth_sim" filename="libgazebo_ros_p3d.so">
             <updateRate>100.0</updateRate>
-            <bodyName>base_link</bodyName>
-            <topicName>/bebop/odom</topicName>
+            <bodyName>${prefix}base_link</bodyName>
+            <topicName>odom</topicName>
             <gaussianNoise>0.0</gaussianNoise>
             <frameName>$(arg world_frame)</frameName>
           </plugin>
         </gazebo>
-    <gazebo reference="sensor_laser">
+        <gazebo reference="${prefix}sensor_laser">
       <sensor type="ray" name="head_hokuyo_sensor">
       <pose>0 0 0 0 0 0</pose>
@@ -76,6 +79,6 @@
       </ray>
       <plugin name="gazebo_ros_head_hokuyo_controller" filename="libgazebo_ros_laser.so">
-        <topicName>/bebop/laser_scan</topicName>
-        <frameName>sensor_laser</frameName>
+        <topicName>laser_scan</topicName>
+        <frameName>${prefix}sensor_laser</frameName>
       </plugin>
     </sensor>

Commit message: added the ouster lidar

File: bebop_gazebo/urdf/bebop.urdf.xacro (robot description, xacro)
@@ -16,27 +16,7 @@
   <xacro:property name="laz_radius" value="0.04"/>
   <xacro:property name="laz_height" value="0.1"/>
-  <!--Laser Scan-->
-  <link name="sensor_laser">
-    <visual>
-      <geometry>
-        <mesh filename="package://bebop_gazebo/meshes/hokuyo.dae"/>
-        <!--box size="${laser_size_x} ${laser_size_y} ${laser_size_z}"/-->
-      </geometry>
-      <material name="blue"/>
-    </visual>
-    <collision>
-      <geometry>
-        <box size="${laser_size_x} ${laser_size_y} ${laser_size_z}"/>
-      </geometry>
-    </collision>
-    <inertial>
-      <mass value="0.00000000001"/>
-      <inertia ixx="${(1/12) * 0.1 * (3 * base_radius * base_radius + base_height * base_height)}" ixy="0" ixz="0" iyy="${(1/12) * 0.1 * (3 * base_radius * base_radius + base_height * base_height)}" iyz="0" izz="${(1/2) * 0.1 * base_radius * base_radius}"/>
-    </inertial>
-  </link>
-  <joint name="sensor_laser_joint" type="fixed">
-    <origin xyz="${laser_origin_x} ${laser_origin_y} ${laser_origin_z}" rpy="0 0 0" />
-    <parent link="base_link"/>
-    <child link="sensor_laser" />
-  </joint>
+  <xacro:include filename="$(find ouster_os1_64)/urdf/os1_64.urdf.xacro"/>
+  <xacro:os1_64 parent="base" name="ouster" prefix="/os1_cloud_node" hz="10" samples="512">
+    <origin xyz="0 0 0" rpy="0 0 0" />
+  </xacro:os1_64>
 </robot>

Commit message: updated

File: bebop_gazebo/urdf/bebop.urdf.xacro (robot description, xacro)
@@ -18,5 +18,5 @@
   <xacro:include filename="$(find ouster_os1_64)/urdf/os1_64.urdf.xacro"/>
   <xacro:os1_64 parent="base" name="ouster" prefix="/os1_cloud_node" hz="10" samples="512">
-    <origin xyz="0 0 0" rpy="0 0 0" />
+    <origin xyz="0 0 0.05" rpy="0 0 0" />
   </xacro:os1_64>
 </robot>

Commit message: added velodyne lidar

File: bebop_gazebo/urdf/bebop.urdf.xacro (robot description, xacro)
@@ -16,7 +16,7 @@
   <xacro:property name="laz_radius" value="0.04"/>
   <xacro:property name="laz_height" value="0.1"/>
-  <xacro:include filename="$(find ouster_os1_64)/urdf/os1_64.urdf.xacro"/>
-  <xacro:os1_64 parent="base" name="ouster" prefix="/os1_cloud_node" hz="10" samples="512">
-    <origin xyz="0 0 0.05" rpy="0 0 0" />
-  </xacro:os1_64>
+  <xacro:include filename="$(find velodyne_description)/urdf/VLP-16.urdf.xacro"/>
+  <xacro:VLP-16 parent="base_link" name="velodyne" topic="/velodyne_points" hz="50" samples="440" gpu="true">
+    <origin xyz="0 0 0.04" rpy="0 0 0" />
+  </xacro:VLP-16>
 </robot>
